File: Wheel-Control-Board/Wheel-Control-Board-Design/BoardV1Proto/BoardV1Proto.kicad_sch (KiCad schematic)
At the start: 8 parts

Commit message: Did some work on board file
Parts:
- removed R?: R, symbol Device:R
- removed SW?: SW_Push, symbol Switch:SW_Push
- added R? (x3): R, symbol Device:R
- added RV? (x2): R_Potentiometer, symbol Device:R_Potentiometer
- added SW? (x3): SW_Push, symbol Switch:SW_Push
Connections:
- net +3V3: now also R?.2, R?.2, R?.2, RV?.1, RV?.1, SW?.2, SW?.2, SW?.2
- net GND: now also R?.1, R?.1, R?.1, RV?.3, RV?.3
- net at U?.16 (IO13): now also SW?.1
- net at U?.23 (IO15): now also SW?.1
- net at U?.24 (IO2): now also SW?.1
- net at U?.25 (IO0): now also RV?.2
- net at U?.26 (IO4): now also RV?.2
- net VCC: now reaches BT?.1 (+)
